File: Solar_Actuators/Solar Panels Rev1/Solar Cell Y/+Y/v3_SolarCellX/SolarCell+Y.sch (KiCad schematic (older format))
At the start: 28 parts, among them IC1 symbols_TSL2561, J1 symbols_XF2M-1015-1A, J2 U.FL-R-SMT-1, Q1 IRLML2803, U1 HHM17139B2, U2 NDS8434

Commit message: Comitting again!
Parts:
- Q1: symbol SolarCellZ_v1-rescue:IRLML2803TRPBF-mainboard-misc-circuits-rescue -> SolarCell+Y-rescue:IRLML2803TRPBF-mainboard-misc-circuits-rescue-SolarCellZ_v1-rescue
- R5, R6, R7: symbol SolarCellZ_v1-rescue:RESISTOR0603-mainboard-misc-circuits-rescue -> SolarCell+Y-rescue:RESISTOR0603-mainboard-misc-circuits-rescue-SolarCellZ_v1-rescue
- U2: symbol SolarCellZ_v1-rescue:NDS8434-symbols-misc-circuits-rescue -> SolarCell+Y-rescue:NDS8434-symbols-misc-circuits-rescue-SolarCellZ_v1-rescue
Changed lines of the file:
@@
 EESchema Schematic File Version 4
 LIBS:SolarCell+Y-cache
-LIBS:SolarCellZ_v1-cache
 EELAYER 30 0
 EELAYER END
@@
 	8800 5100 9150 5100
 $Comp
-L SolarCellZ_v1-rescue:RESISTOR0603-mainboard-misc-circuits-rescue R7
+L SolarCell+Y-rescue:RESISTOR0603-mainboard-misc-circuits-rescue-SolarCellZ_v1-rescue R7
 U 1 1 5DB28BB7
 P 8800 5300
@@
 $EndComp
 $Comp
-L SolarCellZ_v1-rescue:RESISTOR0603-mainboard-misc-circuits-rescue R5
+L SolarCell+Y-rescue:RESISTOR0603-mainboard-misc-circuits-rescue-SolarCellZ_v1-rescue R5
 U 1 1 5DB28BC9
 P 8100 5400
@@
 $EndComp
 $Comp
-L SolarCellZ_v1-rescue:RESISTOR0603-mainboard-misc-circuits-rescue R6
+L SolarCell+Y-rescue:RESISTOR0603-mainboard-misc-circuits-rescue-SolarCellZ_v1-rescue R6
 U 1 1 5DB28BCF
 P 8300 5200
@@
 $EndComp
 $Comp
-L SolarCellZ_v1-rescue:IRLML2803TRPBF-mainboard-misc-circuits-rescue Q1
+L SolarCell+Y-rescue:IRLML2803TRPBF-mainboard-misc-circuits-rescue-SolarCellZ_v1-rescue Q1
 U 1 1 5DB28BE3
 P 8600 5500
@@
 $EndComp
 $Comp
-L SolarCellZ_v1-rescue:NDS8434-symbols-misc-circuits-rescue U?
+L SolarCell+Y-rescue:NDS8434-symbols-misc-circuits-rescue-SolarCellZ_v1-rescue U?
 U 1 1 5DB28C34
 P 9650 5400
